File: Small_CKT/Small_CKT.kicad_sch (KiCad schematic)
At the start: 5 parts, among them SW1 SW_Push

Commit message: Added footprints to LED, SW, and battery
Parts:
- BT1, BT2: footprint (none) -> Connector_Molex:Molex_Mega-Fit_76829-0002_2x01_P5.70mm_Vertical
- D1, D3: footprint (none) -> LED_THT:LED_D5.0mm_Clear
- SW1: footprint (none) -> Button_Switch_THT:SW_PUSH_6mm
Changed lines of the file:
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@@
       (effects (font (size 1.27 1.27)) (justify left))
     )
-    (property "Footprint" "" (at 80.01 104.14 0)
+    (property "Footprint" "LED_THT:LED_D5.0mm_Clear" (at 80.01 104.14 0)
       (effects (font (size 1.27 1.27)) hide)
     )
@@
       (effects (font (size 1.27 1.27)) (justify left))
     )
-    (property "Footprint" "" (at 96.52 104.14 0)
+    (property "Footprint" "LED_THT:LED_D5.0mm_Clear" (at 96.52 104.14 0)
       (effects (font (size 1.27 1.27)) hide)
     )
@@
       (effects (font (size 1.27 1.27)))
     )
-    (property "Footprint" "" (at 113.03 85.09 0)
+    (property "Footprint" "Button_Switch_THT:SW_PUSH_6mm" (at 113.03 85.09 0)
       (effects (font (size 1.27 1.27)) hide)
     )
@@
       (effects (font (size 1.27 1.27)) (justify left))
     )
-    (property "Footprint" "" (at 134.62 102.616 90)
+    (property "Footprint" "Connector_Molex:Molex_Mega-Fit_76829-0002_2x01_P5.70mm_Vertical" (at 134.62 102.616 90)
       (effects (font (size 1.27 1.27)) hide)
     )
@@
       (effects (font (size 1.27 1.27)) (justify left))
     )
-    (property "Footprint" "" (at 158.75 102.616 90)
+    (property "Footprint" "Connector_Molex:Molex_Mega-Fit_76829-0002_2x01_P5.70mm_Vertical" (at 158.75 102.616 90)
       (effects (font (size 1.27 1.27)) hide)
     )
